File: PCB/FPGA.sch (KiCad schematic (older format))
At the start: 5 parts, among them J5 TSM-105-01-S-DV, U2 S25FL128SAGMFI000, X1 SG-5032CAN

Commit message: Initial commit of the Quartus project
Connections:
- net labels added: Motor_PWM_1, Motor_PWM_2
- net labels removed: Motor_PWM_N, Motor_PWM_P
Changed lines of the file:
@@
 	9000 5000 9500 5000
 Text HLabel 9500 5100 2    50   Output ~ 0
-Motor_PWM_N
+Motor_PWM_2
 Text HLabel 9500 5000 2    50   Output ~ 0
-Motor_PWM_P
+Motor_PWM_1
 Text Notes 950  6750 0    197  ~ 0
 TODO:\n- Cyclone 10 (10CL016YE144C8G)\n- JTAG pull-up / down resistors\n- Config signals\n- Connect I/Os (and double-check)
