File: PCB/LightSensor.sch (KiCad schematic (older format))
At the start: 5 parts, among them U4 VEML6035

Commit message: Add the FPGA symbol
Parts:
- renumbered C13 to C11, U4 to U3
Changed lines of the file:
@@
 $Descr A4 11693 8268
 encoding utf-8
-Sheet 17 17
+Sheet 17 19
 Title "Litter Robot 3 - Ambient light sensor"
 Date "2021-03-20"
@@
 $EndDescr
 $Comp
-L LitterRobot:VEML6035 U4
+L LitterRobot:VEML6035 U3
 U 1 1 6062B3AA
 P 5150 3750
-F 0 "U4" H 4806 3796 50  0000 R CNN
+F 0 "U3" H 4806 3796 50  0000 R CNN
 F 1 "VEML6035" H 4806 3705 50  0000 R CNN
 F 2 "LitterRobot:Vishay_VEML6035" H 5150 3250 50  0001 C CNN
@@
 P 5250 4250
 AR Path="/6062F82F" Ref="#PWR?"  Part="1"
-AR Path="/60624089/6062F82F" Ref="#PWR075"  Part="1"
-F 0 "#PWR075" H 5250 4000 50  0001 C CNN
+AR Path="/60624089/6062F82F" Ref="#PWR068"  Part="1"
+F 0 "#PWR068" H 5250 4000 50  0001 C CNN
 F 1 "GND" H 5255 4077 50  0000 C CNN
 F 2 "" H 5250 4250 50  0001 C CNN
@@
 P 5250 3250
 AR Path="/6062F849" Ref="#PWR?"  Part="1"
-AR Path="/60624089/6062F849" Ref="#PWR074"  Part="1"
-F 0 "#PWR074" H 5250 3100 50  0001 C CNN
+AR Path="/60624089/6062F849" Ref="#PWR067"  Part="1"
+F 0 "#PWR067" H 5250 3100 50  0001 C CNN
 F 1 "+3V3" H 5265 3423 50  0000 C CNN
 F 2 "" H 5250 3250 50  0001 C CNN
@@
 P 6000 2900
 AR Path="/60633A13" Ref="#PWR?"  Part="1"
-AR Path="/60624089/60633A13" Ref="#PWR076"  Part="1"
-F 0 "#PWR076" H 6000 2750 50  0001 C CNN
+AR Path="/60624089/60633A13" Ref="#PWR069"  Part="1"
+F 0 "#PWR069" H 6000 2750 50  0001 C CNN
 F 1 "+3V3" H 6015 3073 50  0000 C CNN
 F 2 "" H 6000 2900 50  0001 C CNN
@@
 P 4000 3750
 AR Path="/603F20AB/606362ED" Ref="C?"  Part="1"
-AR Path="/60624089/606362ED" Ref="C13"  Part="1"
-F 0 "C13" H 4115 3841 50  0000 L CNN
+AR Path="/60624089/606362ED" Ref="C11"  Part="1"
+F 0 "C11" H 4115 3841 50  0000 L CNN
 F 1 "100nF" H 4115 3750 50  0000 L CNN
 F 2 "Capacitor_SMD:C_0603_1608Metric" H 4038 3600 50  0001 C CNN

Commit message: Connect the FPGA configuration signals
Parts:
- C11: Part_Number C1608X5R1H104K080AA -> (none); Part_number (none) -> C1608X5R1H104K080AA
- R39: renamed from R40; Part_Number CR0603-FX-3301ELF -> (none); Part_number (none) -> CR0603-FX-3301ELF
- R40: renamed from R41; Part_Number CR0603-FX-3301ELF -> (none); Part_number (none) -> CR0603-FX-3301ELF
- R41: renamed from R42; Part_Number CR0603-FX-3301ELF -> (none); Part_number (none) -> CR0603-FX-3301ELF
Changed lines of the file:
@@
 $Descr A4 11693 8268
 encoding utf-8
-Sheet 17 19
+Sheet 16 19
 Title "Litter Robot 3 - Ambient light sensor"
 Date "2021-03-20"
@@
 P 5250 4250
 AR Path="/6062F82F" Ref="#PWR?"  Part="1"
-AR Path="/60624089/6062F82F" Ref="#PWR068"  Part="1"
-F 0 "#PWR068" H 5250 4000 50  0001 C CNN
+AR Path="/60624089/6062F82F" Ref="#PWR067"  Part="1"
+F 0 "#PWR067" H 5250 4000 50  0001 C CNN
 F 1 "GND" H 5255 4077 50  0000 C CNN
 F 2 "" H 5250 4250 50  0001 C CNN
@@
 P 5250 3250
 AR Path="/6062F849" Ref="#PWR?"  Part="1"
-AR Path="/60624089/6062F849" Ref="#PWR067"  Part="1"
-F 0 "#PWR067" H 5250 3100 50  0001 C CNN
+AR Path="/60624089/6062F849" Ref="#PWR066"  Part="1"
+F 0 "#PWR066" H 5250 3100 50  0001 C CNN
 F 1 "+3V3" H 5265 3423 50  0000 C CNN
 F 2 "" H 5250 3250 50  0001 C CNN
@@
 AR Path="/603F20AB/60632EF7" Ref="R?"  Part="1"
 AR Path="/603F1DCE/60632EF7" Ref="R?"  Part="1"
-AR Path="/60624089/60632EF7" Ref="R40"  Part="1"
-F 0 "R40" H 6070 3296 50  0000 L CNN
+AR Path="/60624089/60632EF7" Ref="R39"  Part="1"
+F 0 "R39" H 6070 3296 50  0000 L CNN
 F 1 "3.3k" H 6070 3205 50  0000 L CNN
 F 2 "Resistor_SMD:R_0603_1608Metric" V 5930 3250 50  0001 C CNN
-F 3 "~" H 6000 3250 50  0001 C CNN
-F 4 "CR0603-FX-3301ELF" H 6000 3250 50  0001 C CNN "Part_Number"
+F 3 "https://www.bourns.com/docs/product-datasheets/CRxxxxx.pdf" H 6000 3250 50  0001 C CNN
+F 4 "" H 6000 3250 50  0001 C CNN "Part_Number"
+F 5 "CR0603-FX-3301ELF" H 6000 3250 50  0001 C CNN "Part_number"
 	1    6000 3250
 	1    0    0    -1
@@
 AR Path="/603F20AB/60632F30" Ref="R?"  Part="1"
 AR Path="/603F1DCE/60632F30" Ref="R?"  Part="1"
-AR Path="/60624089/60632F30" Ref="R41"  Part="1"
-F 0 "R41" H 6570 3296 50  0000 L CNN
+AR Path="/60624089/60632F30" Ref="R40"  Part="1"
+F 0 "R40" H 6570 3296 50  0000 L CNN
 F 1 "3.3k" H 6570 3205 50  0000 L CNN
 F 2 "Resistor_SMD:R_0603_1608Metric" V 6430 3250 50  0001 C CNN
-F 3 "~" H 6500 3250 50  0001 C CNN
-F 4 "CR0603-FX-3301ELF" H 6500 3250 50  0001 C CNN "Part_Number"
+F 3 "https://www.bourns.com/docs/product-datasheets/CRxxxxx.pdf" H 6500 3250 50  0001 C CNN
+F 4 "" H 6500 3250 50  0001 C CNN "Part_Number"
+F 5 "CR0603-FX-3301ELF" H 6500 3250 50  0001 C CNN "Part_number"
 	1    6500 3250
 	1    0    0    -1
@@
 AR Path="/603F20AB/60633461" Ref="R?"  Part="1"
 AR Path="/603F1DCE/60633461" Ref="R?"  Part="1"
-AR Path="/60624089/60633461" Ref="R42"  Part="1"
-F 0 "R42" H 7070 3296 50  0000 L CNN
+AR Path="/60624089/60633461" Ref="R41"  Part="1"
+F 0 "R41" H 7070 3296 50  0000 L CNN
 F 1 "3.3k" H 7070 3205 50  0000 L CNN
 F 2 "Resistor_SMD:R_0603_1608Metric" V 6930 3250 50  0001 C CNN
-F 3 "~" H 7000 3250 50  0001 C CNN
-F 4 "CR0603-FX-3301ELF" H 7000 3250 50  0001 C CNN "Part_Number"
+F 3 "https://www.bourns.com/docs/product-datasheets/CRxxxxx.pdf" H 7000 3250 50  0001 C CNN
+F 4 "" H 7000 3250 50  0001 C CNN "Part_Number"
+F 5 "CR0603-FX-3301ELF" H 7000 3250 50  0001 C CNN "Part_number"
 	1    7000 3250
 	1    0    0    -1
@@
 P 6000 2900
 AR Path="/60633A13" Ref="#PWR?"  Part="1"
-AR Path="/60624089/60633A13" Ref="#PWR069"  Part="1"
-F 0 "#PWR069" H 6000 2750 50  0001 C CNN
+AR Path="/60624089/60633A13" Ref="#PWR068"  Part="1"
+F 0 "#PWR068" H 6000 2750 50  0001 C CNN
 F 1 "+3V3" H 6015 3073 50  0000 C CNN
 F 2 "" H 6000 2900 50  0001 C CNN
@@
 F 2 "Capacitor_SMD:C_0603_1608Metric" H 4038 3600 50  0001 C CNN
 F 3 "~" H 4000 3750 50  0001 C CNN
-F 4 "C1608X5R1H104K080AA" H 4000 3750 50  0001 C CNN "Part_Number"
+F 4 "" H 4000 3750 50  0001 C CNN "Part_Number"
 F 5 "50V" H 4115 3659 50  0000 L CNN "Voltage"
+F 6 "C1608X5R1H104K080AA" H 4000 3750 50  0001 C CNN "Part_number"
 	1    4000 3750
 	1    0    0    -1
