File: PCB/LightSensor.sch (KiCad schematic (older format))
At the start: 5 parts, among them U3 VEML6035

Commit message: Add support for the weight sensor
Parts:
- renumbered R39 to R41, R40 to R42, R41 to R43
Changed lines of the file:
@@
 $Descr A4 11693 8268
 encoding utf-8
-Sheet 16 19
+Sheet 16 20
 Title "Litter Robot 3 - Ambient light sensor"
-Date "2021-03-28"
+Date "2021-04-02"
 Rev "A1"
 Comp "L. Sartory"
@@
 P 5250 4250
 AR Path="/6062F82F" Ref="#PWR?"  Part="1"
-AR Path="/60624089/6062F82F" Ref="#PWR067"  Part="1"
-F 0 "#PWR067" H 5250 4000 50  0001 C CNN
+AR Path="/60624089/6062F82F" Ref="#PWR069"  Part="1"
+F 0 "#PWR069" H 5250 4000 50  0001 C CNN
 F 1 "GND" H 5255 4077 50  0000 C CNN
 F 2 "" H 5250 4250 50  0001 C CNN
@@
 P 5250 3250
 AR Path="/6062F849" Ref="#PWR?"  Part="1"
-AR Path="/60624089/6062F849" Ref="#PWR066"  Part="1"
-F 0 "#PWR066" H 5250 3100 50  0001 C CNN
+AR Path="/60624089/6062F849" Ref="#PWR068"  Part="1"
+F 0 "#PWR068" H 5250 3100 50  0001 C CNN
 F 1 "+3V3" H 5265 3423 50  0000 C CNN
 F 2 "" H 5250 3250 50  0001 C CNN
@@
 AR Path="/603F20AB/60632EF7" Ref="R?"  Part="1"
 AR Path="/603F1DCE/60632EF7" Ref="R?"  Part="1"
-AR Path="/60624089/60632EF7" Ref="R39"  Part="1"
-F 0 "R39" H 6070 3296 50  0000 L CNN
+AR Path="/60624089/60632EF7" Ref="R41"  Part="1"
+F 0 "R41" H 6070 3296 50  0000 L CNN
 F 1 "3.3k" H 6070 3205 50  0000 L CNN
 F 2 "Resistor_SMD:R_0603_1608Metric" V 5930 3250 50  0001 C CNN
@@
 AR Path="/603F20AB/60632F30" Ref="R?"  Part="1"
 AR Path="/603F1DCE/60632F30" Ref="R?"  Part="1"
-AR Path="/60624089/60632F30" Ref="R40"  Part="1"
-F 0 "R40" H 6570 3296 50  0000 L CNN
+AR Path="/60624089/60632F30" Ref="R42"  Part="1"
+F 0 "R42" H 6570 3296 50  0000 L CNN
 F 1 "3.3k" H 6570 3205 50  0000 L CNN
 F 2 "Resistor_SMD:R_0603_1608Metric" V 6430 3250 50  0001 C CNN
@@
 AR Path="/603F20AB/60633461" Ref="R?"  Part="1"
 AR Path="/603F1DCE/60633461" Ref="R?"  Part="1"
-AR Path="/60624089/60633461" Ref="R41"  Part="1"
-F 0 "R41" H 7070 3296 50  0000 L CNN
+AR Path="/60624089/60633461" Ref="R43"  Part="1"
+F 0 "R43" H 7070 3296 50  0000 L CNN
 F 1 "3.3k" H 7070 3205 50  0000 L CNN
 F 2 "Resistor_SMD:R_0603_1608Metric" V 6930 3250 50  0001 C CNN
@@
 P 6000 2900
 AR Path="/60633A13" Ref="#PWR?"  Part="1"
-AR Path="/60624089/60633A13" Ref="#PWR068"  Part="1"
-F 0 "#PWR068" H 6000 2750 50  0001 C CNN
+AR Path="/60624089/60633A13" Ref="#PWR070"  Part="1"
+F 0 "#PWR070" H 6000 2750 50  0001 C CNN
 F 1 "+3V3" H 6015 3073 50  0000 C CNN
 F 2 "" H 6000 2900 50  0001 C CNN

Commit message: Re-annotate all components
Parts:
- renumbered C11 to C32, R41 to R28, R42 to R29, R43 to R30, U3 to U6
Changed lines of the file:
@@
 $Descr A4 11693 8268
 encoding utf-8
-Sheet 16 22
+Sheet 9 22
 Title "Litter Robot 3 - Ambient light sensor"
-Date "2021-04-03"
+Date "2021-04-05"
 Rev "A1"
 Comp "L. Sartory"
@@
 $EndDescr
 $Comp
-L LitterRobot:VEML6035 U3
+L LitterRobot:VEML6035 U6
 U 1 1 6062B3AA
 P 5150 3750
-F 0 "U3" H 4806 3796 50  0000 R CNN
+F 0 "U6" H 4806 3796 50  0000 R CNN
 F 1 "VEML6035" H 4806 3705 50  0000 R CNN
 F 2 "LitterRobot:Vishay_VEML6035" H 5150 3250 50  0001 C CNN
@@
 P 5250 4250
 AR Path="/6062F82F" Ref="#PWR?"  Part="1"
-AR Path="/60624089/6062F82F" Ref="#PWR069"  Part="1"
-F 0 "#PWR069" H 5250 4000 50  0001 C CNN
+AR Path="/60624089/6062F82F" Ref="#PWR081"  Part="1"
+F 0 "#PWR081" H 5250 4000 50  0001 C CNN
 F 1 "GND" H 5255 4077 50  0000 C CNN
 F 2 "" H 5250 4250 50  0001 C CNN
@@
 P 5250 3250
 AR Path="/6062F849" Ref="#PWR?"  Part="1"
-AR Path="/60624089/6062F849" Ref="#PWR068"  Part="1"
-F 0 "#PWR068" H 5250 3100 50  0001 C CNN
+AR Path="/60624089/6062F849" Ref="#PWR080"  Part="1"
+F 0 "#PWR080" H 5250 3100 50  0001 C CNN
 F 1 "+3V3" H 5265 3423 50  0000 C CNN
 F 2 "" H 5250 3250 50  0001 C CNN
@@
 AR Path="/603F20AB/60632EF7" Ref="R?"  Part="1"
 AR Path="/603F1DCE/60632EF7" Ref="R?"  Part="1"
-AR Path="/60624089/60632EF7" Ref="R41"  Part="1"
-F 0 "R41" H 6070 3296 50  0000 L CNN
+AR Path="/60624089/60632EF7" Ref="R28"  Part="1"
+F 0 "R28" H 6070 3296 50  0000 L CNN
 F 1 "3.3k" H 6070 3205 50  0000 L CNN
 F 2 "Resistor_SMD:R_0603_1608Metric" V 5930 3250 50  0001 C CNN
@@
 AR Path="/603F20AB/60632F30" Ref="R?"  Part="1"
 AR Path="/603F1DCE/60632F30" Ref="R?"  Part="1"
-AR Path="/60624089/60632F30" Ref="R42"  Part="1"
-F 0 "R42" H 6570 3296 50  0000 L CNN
+AR Path="/60624089/60632F30" Ref="R29"  Part="1"
+F 0 "R29" H 6570 3296 50  0000 L CNN
 F 1 "3.3k" H 6570 3205 50  0000 L CNN
 F 2 "Resistor_SMD:R_0603_1608Metric" V 6430 3250 50  0001 C CNN
@@
 AR Path="/603F20AB/60633461" Ref="R?"  Part="1"
 AR Path="/603F1DCE/60633461" Ref="R?"  Part="1"
-AR Path="/60624089/60633461" Ref="R43"  Part="1"
-F 0 "R43" H 7070 3296 50  0000 L CNN
+AR Path="/60624089/60633461" Ref="R30"  Part="1"
+F 0 "R30" H 7070 3296 50  0000 L CNN
 F 1 "3.3k" H 7070 3205 50  0000 L CNN
 F 2 "Resistor_SMD:R_0603_1608Metric" V 6930 3250 50  0001 C CNN
@@
 P 6000 2900
 AR Path="/60633A13" Ref="#PWR?"  Part="1"
-AR Path="/60624089/60633A13" Ref="#PWR070"  Part="1"
-F 0 "#PWR070" H 6000 2750 50  0001 C CNN
+AR Path="/60624089/60633A13" Ref="#PWR079"  Part="1"
+F 0 "#PWR079" H 6000 2750 50  0001 C CNN
 F 1 "+3V3" H 6015 3073 50  0000 C CNN
 F 2 "" H 6000 2900 50  0001 C CNN
@@
 P 4000 3750
 AR Path="/603F20AB/606362ED" Ref="C?"  Part="1"
-AR Path="/60624089/606362ED" Ref="C11"  Part="1"
-F 0 "C11" H 4115 3841 50  0000 L CNN
+AR Path="/60624089/606362ED" Ref="C32"  Part="1"
+F 0 "C32" H 4115 3841 50  0000 L CNN
 F 1 "100nF" H 4115 3750 50  0000 L CNN
 F 2 "Capacitor_SMD:C_0603_1608Metric" H 4038 3600 50  0001 C CNN

Commit message: Add the EMB1061 Bluetooth module
Parts:
- renumbered U6 to U7
Changed lines of the file:
@@
 $Descr A4 11693 8268
 encoding utf-8
-Sheet 9 22
+Sheet 9 23
 Title "Litter Robot 3 - Ambient light sensor"
-Date "2021-04-05"
+Date "2021-04-10"
 Rev "A1"
 Comp "L. Sartory"
@@
 $EndDescr
 $Comp
-L LitterRobot:VEML6035 U6
+L LitterRobot:VEML6035 U7
 U 1 1 6062B3AA
 P 5150 3750
-F 0 "U6" H 4806 3796 50  0000 R CNN
+F 0 "U7" H 4806 3796 50  0000 R CNN
 F 1 "VEML6035" H 4806 3705 50  0000 R CNN
 F 2 "LitterRobot:Vishay_VEML6035" H 5150 3250 50  0001 C CNN
@@
 P 5250 4250
 AR Path="/6062F82F" Ref="#PWR?"  Part="1"
-AR Path="/60624089/6062F82F" Ref="#PWR081"  Part="1"
-F 0 "#PWR081" H 5250 4000 50  0001 C CNN
+AR Path="/60624089/6062F82F" Ref="#PWR084"  Part="1"
+F 0 "#PWR084" H 5250 4000 50  0001 C CNN
 F 1 "GND" H 5255 4077 50  0000 C CNN
 F 2 "" H 5250 4250 50  0001 C CNN
@@
 P 5250 3250
 AR Path="/6062F849" Ref="#PWR?"  Part="1"
-AR Path="/60624089/6062F849" Ref="#PWR080"  Part="1"
-F 0 "#PWR080" H 5250 3100 50  0001 C CNN
+AR Path="/60624089/6062F849" Ref="#PWR083"  Part="1"
+F 0 "#PWR083" H 5250 3100 50  0001 C CNN
 F 1 "+3V3" H 5265 3423 50  0000 C CNN
 F 2 "" H 5250 3250 50  0001 C CNN
@@
 P 6000 2900
 AR Path="/60633A13" Ref="#PWR?"  Part="1"
-AR Path="/60624089/60633A13" Ref="#PWR079"  Part="1"
-F 0 "#PWR079" H 6000 2750 50  0001 C CNN
+AR Path="/60624089/60633A13" Ref="#PWR082"  Part="1"
+F 0 "#PWR082" H 6000 2750 50  0001 C CNN
 F 1 "+3V3" H 6015 3073 50  0000 C CNN
 F 2 "" H 6000 2900 50  0001 C CNN

Commit message: Add jumpers on the power supply outputs
Parts:
- renumbered R28 to R32, R29 to R33, R30 to R34
Changed lines of the file:
@@
 Sheet 10 23
 Title "Litter Robot 3 - Ambient light sensor"
-Date "2021-04-10"
+Date "2021-05-24"
 Rev "A1"
 Comp "L. Sartory"
@@
 AR Path="/603F20AB/60632EF7" Ref="R?"  Part="1"
 AR Path="/603F1DCE/60632EF7" Ref="R?"  Part="1"
-AR Path="/60624089/60632EF7" Ref="R28"  Part="1"
-F 0 "R28" H 6070 3296 50  0000 L CNN
+AR Path="/60624089/60632EF7" Ref="R32"  Part="1"
+F 0 "R32" H 6070 3296 50  0000 L CNN
 F 1 "3.3k" H 6070 3205 50  0000 L CNN
 F 2 "Resistor_SMD:R_0603_1608Metric" V 5930 3250 50  0001 C CNN
@@
 AR Path="/603F20AB/60632F30" Ref="R?"  Part="1"
 AR Path="/603F1DCE/60632F30" Ref="R?"  Part="1"
-AR Path="/60624089/60632F30" Ref="R29"  Part="1"
-F 0 "R29" H 6570 3296 50  0000 L CNN
+AR Path="/60624089/60632F30" Ref="R33"  Part="1"
+F 0 "R33" H 6570 3296 50  0000 L CNN
 F 1 "3.3k" H 6570 3205 50  0000 L CNN
 F 2 "Resistor_SMD:R_0603_1608Metric" V 6430 3250 50  0001 C CNN
@@
 AR Path="/603F20AB/60633461" Ref="R?"  Part="1"
 AR Path="/603F1DCE/60633461" Ref="R?"  Part="1"
-AR Path="/60624089/60633461" Ref="R30"  Part="1"
-F 0 "R30" H 7070 3296 50  0000 L CNN
+AR Path="/60624089/60633461" Ref="R34"  Part="1"
+F 0 "R34" H 7070 3296 50  0000 L CNN
 F 1 "3.3k" H 7070 3205 50  0000 L CNN
 F 2 "Resistor_SMD:R_0603_1608Metric" V 6930 3250 50  0001 C CNN
