File: PCB/PushButtonDual.sch (KiCad schematic (older format))
At the start: 3 parts, among them SW3 PCB_Push_Button, SW4 PCB_Push_Button

Commit message: Connect the FPGA configuration signals
Parts:
- R21: Part_Number CR0603-FX-1002ELF -> (none); Part_number (none) -> CR0603-FX-1002ELF
Changed lines of the file:
@@
 F 1 "10k" H 5070 3955 50  0000 L CNN
 F 2 "Resistor_SMD:R_0603_1608Metric" V 4930 4000 50  0001 C CNN
-F 3 "~" H 5000 4000 50  0001 C CNN
-F 4 "CR0603-FX-1002ELF" H 5000 4000 50  0001 C CNN "Part_Number"
+F 3 "https://www.bourns.com/docs/product-datasheets/CRxxxxx.pdf" H 5000 4000 50  0001 C CNN
+F 4 "" H 5000 4000 50  0001 C CNN "Part_Number"
+F 5 "CR0603-FX-1002ELF" H 5000 4000 50  0001 C CNN "Part_number"
 	1    5000 4000
 	1    0    0    -1
