File: PCB/RgbLed.sch (KiCad schematic (older format))
At the start: 7 parts, among them Q1 BC817, Q2 BC817, Q3 BC817

Commit message: Connect the FPGA configuration signals
Parts:
- D1: Part_Number SMLVN6RGB1U1 -> (none); Part_number (none) -> SMLVN6RGB1U1
- Q1, Q2, Q3: Part_Number BC817-25,215 -> (none); Part_number (none) -> BC817-25,215
- R1: Part_Number CR0603-FX-1780ELF -> (none); Part_number (none) -> CR0603-FX-1780ELF
- R2, R3: Part_Number CR0603-FX-2210ELF -> (none); Part_number (none) -> CR0603-FX-2210ELF
Changed lines of the file:
@@
 $Descr A4 11693 8268
 encoding utf-8
-Sheet 8 19
+Sheet 3 19
 Title "Litter Robot 3 - RGB LED"
 Date "2021-02-28"
@@
 F 2 "Package_TO_SOT_SMD:SOT-23" H 4100 4125 50  0001 L CIN
 F 3 "https://www.onsemi.com/pub/Collateral/BC818-D.pdf" H 3900 4200 50  0001 L CNN
-F 4 "BC817-25,215" H 3900 4200 50  0001 C CNN "Part_Number"
+F 4 "" H 3900 4200 50  0001 C CNN "Part_Number"
+F 5 "BC817-25,215" H 3900 4200 50  0001 C CNN "Part_number"
 	1    3900 4200
 	1    0    0    -1
@@
 F 1 "178R" H 4070 4605 50  0000 L CNN
 F 2 "Resistor_SMD:R_0603_1608Metric" V 3930 4650 50  0001 C CNN
-F 3 "~" H 4000 4650 50  0001 C CNN
-F 4 "CR0603-FX-1780ELF" H 4000 4650 50  0001 C CNN "Part_Number"
+F 3 "https://www.bourns.com/docs/product-datasheets/CRxxxxx.pdf" H 4000 4650 50  0001 C CNN
+F 4 "" H 4000 4650 50  0001 C CNN "Part_Number"
+F 5 "CR0603-FX-1780ELF" H 4000 4650 50  0001 C CNN "Part_number"
 	1    4000 4650
 	1    0    0    -1
@@
 F 2 "LitterRobot:ROHM_SMLVN6" H 5500 2850 50  0001 C CNN
 F 3 "https://fscdn.rohm.com/en/products/databook/datasheet/opto/led/chip_multi/smlvn6rgb1w-e.pdf" H 5500 3150 50  0001 C CNN
-F 4 "SMLVN6RGB1U1" H 5500 3200 50  0001 C CNN "Part_Number"
+F 4 "" H 5500 3200 50  0001 C CNN "Part_Number"
+F 5 "SMLVN6RGB1U1" H 5500 3200 50  0001 C CNN "Part_number"
 	1    5500 3200
 	0    1    1    0
@@
 F 1 "221R" H 5570 4605 50  0000 L CNN
 F 2 "Resistor_SMD:R_0603_1608Metric" V 5430 4650 50  0001 C CNN
-F 3 "~" H 5500 4650 50  0001 C CNN
-F 4 "CR0603-FX-2210ELF" H 5500 4650 50  0001 C CNN "Part_Number"
+F 3 "https://www.bourns.com/docs/product-datasheets/CRxxxxx.pdf" H 5500 4650 50  0001 C CNN
+F 4 "" H 5500 4650 50  0001 C CNN "Part_Number"
+F 5 "CR0603-FX-2210ELF" H 5500 4650 50  0001 C CNN "Part_number"
 	1    5500 4650
 	1    0    0    -1
@@
 F 1 "221R" H 7070 4605 50  0000 L CNN
 F 2 "Resistor_SMD:R_0603_1608Metric" V 6930 4650 50  0001 C CNN
-F 3 "~" H 7000 4650 50  0001 C CNN
-F 4 "CR0603-FX-2210ELF" H 7000 4650 50  0001 C CNN "Part_Number"
+F 3 "https://www.bourns.com/docs/product-datasheets/CRxxxxx.pdf" H 7000 4650 50  0001 C CNN
+F 4 "" H 7000 4650 50  0001 C CNN "Part_Number"
+F 5 "CR0603-FX-2210ELF" H 7000 4650 50  0001 C CNN "Part_number"
 	1    7000 4650
 	1    0    0    -1
@@
 F 2 "Package_TO_SOT_SMD:SOT-23" H 5600 4125 50  0001 L CIN
 F 3 "https://www.onsemi.com/pub/Collateral/BC818-D.pdf" H 5400 4200 50  0001 L CNN
-F 4 "BC817-25,215" H 5400 4200 50  0001 C CNN "Part_Number"
+F 4 "" H 5400 4200 50  0001 C CNN "Part_Number"
+F 5 "BC817-25,215" H 5400 4200 50  0001 C CNN "Part_number"
 	1    5400 4200
 	1    0    0    -1
@@
 F 2 "Package_TO_SOT_SMD:SOT-23" H 7100 4125 50  0001 L CIN
 F 3 "https://www.onsemi.com/pub/Collateral/BC818-D.pdf" H 6900 4200 50  0001 L CNN
-F 4 "BC817-25,215" H 6900 4200 50  0001 C CNN "Part_Number"
+F 4 "" H 6900 4200 50  0001 C CNN "Part_Number"
+F 5 "BC817-25,215" H 6900 4200 50  0001 C CNN "Part_number"
 	1    6900 4200
 	1    0    0    -1
