File: PCB/RgbLed.sch (KiCad schematic (older format))
At the start: 7 parts, among them Q16 BC817, Q17 BC817, Q18 BC817

Commit message: Route more signals
Changed lines of the file:
@@
 $Descr A4 11693 8268
 encoding utf-8
-Sheet 23 23
+Sheet 22 23
 Title "Litter Robot 3 - RGB LED"
 Date "2021-04-10"
@@
 AR Path="/603F1F4D/605BE11A/603E2469" Ref="Q?"  Part="1"
 AR Path="/603F1F4D/605BE15A/603E2469" Ref="Q?"  Part="1"
-F 0 "Q22" H 4091 4246 50  0000 L CNN
+F 0 "Q19" H 4091 4246 50  0000 L CNN
 F 1 "BC817" H 4091 4155 50  0000 L CNN
 F 2 "Package_TO_SOT_SMD:SOT-23" H 4100 4125 50  0001 L CIN
@@
 AR Path="/603F1F4D/605BE11A/603E246F" Ref="R?"  Part="1"
 AR Path="/603F1F4D/605BE15A/603E246F" Ref="R?"  Part="1"
-F 0 "R54" H 4070 4696 50  0000 L CNN
+F 0 "R51" H 4070 4696 50  0000 L CNN
 F 1 "178R" H 4070 4605 50  0000 L CNN
 F 2 "Resistor_SMD:R_0603_1608Metric" V 3930 4650 50  0001 C CNN
@@
 AR Path="/603F1F4D/605BE11A/603E7162" Ref="D?"  Part="1"
 AR Path="/603F1F4D/605BE15A/603E7162" Ref="D?"  Part="1"
-F 0 "D10" H 5500 3697 50  0000 C CNN
+F 0 "D9" H 5500 3697 50  0000 C CNN
 F 1 "SMLVN6RGB1U" H 5500 3606 50  0000 C CNN
 F 2 "LitterRobot:ROHM_SMLVN6" H 5500 2850 50  0001 C CNN
@@
 AR Path="/603F1F4D/605BE11A/603FCE1E" Ref="R?"  Part="1"
 AR Path="/603F1F4D/605BE15A/603FCE1E" Ref="R?"  Part="1"
-F 0 "R55" H 5570 4696 50  0000 L CNN
+F 0 "R52" H 5570 4696 50  0000 L CNN
 F 1 "221R" H 5570 4605 50  0000 L CNN
 F 2 "Resistor_SMD:R_0603_1608Metric" V 5430 4650 50  0001 C CNN
@@
 AR Path="/603F1F4D/605BE11A/603FDBA6" Ref="R?"  Part="1"
 AR Path="/603F1F4D/605BE15A/603FDBA6" Ref="R?"  Part="1"
-F 0 "R56" H 7070 4696 50  0000 L CNN
+F 0 "R53" H 7070 4696 50  0000 L CNN
 F 1 "221R" H 7070 4605 50  0000 L CNN
 F 2 "Resistor_SMD:R_0603_1608Metric" V 6930 4650 50  0001 C CNN
@@
 AR Path="/603F1F4D/605BE11A/6045060B" Ref="Q?"  Part="1"
 AR Path="/603F1F4D/605BE15A/6045060B" Ref="Q?"  Part="1"
-F 0 "Q23" H 5591 4246 50  0000 L CNN
+F 0 "Q20" H 5591 4246 50  0000 L CNN
 F 1 "BC817" H 5591 4155 50  0000 L CNN
 F 2 "Package_TO_SOT_SMD:SOT-23" H 5600 4125 50  0001 L CIN
@@
 AR Path="/603F1F4D/605BE11A/60450E24" Ref="Q?"  Part="1"
 AR Path="/603F1F4D/605BE15A/60450E24" Ref="Q?"  Part="1"
-F 0 "Q24" H 7091 4246 50  0000 L CNN
+F 0 "Q21" H 7091 4246 50  0000 L CNN
 F 1 "BC817" H 7091 4155 50  0000 L CNN
 F 2 "Package_TO_SOT_SMD:SOT-23" H 7100 4125 50  0001 L CIN

Commit message: Fix invalid / missing part numbers
Parts:
- R48: Part_number CR0603-FX-1780ELF -> CR0603-FX-1780ELF
Changed lines of the file:
@@
 $Descr A4 11693 8268
 encoding utf-8
-Sheet 22 23
+Sheet 19 23
 Title "Litter Robot 3 - RGB LED"
 Date "2021-04-10"
@@
 AR Path="/603F1F4D/605BE11A/603E2469" Ref="Q?"  Part="1"
 AR Path="/603F1F4D/605BE15A/603E2469" Ref="Q?"  Part="1"
-F 0 "Q19" H 4091 4246 50  0000 L CNN
+F 0 "Q10" H 4091 4246 50  0000 L CNN
 F 1 "BC817" H 4091 4155 50  0000 L CNN
 F 2 "Package_TO_SOT_SMD:SOT-23" H 4100 4125 50  0001 L CIN
@@
 AR Path="/603F1F4D/605BE11A/603E246F" Ref="R?"  Part="1"
 AR Path="/603F1F4D/605BE15A/603E246F" Ref="R?"  Part="1"
-F 0 "R51" H 4070 4696 50  0000 L CNN
+F 0 "R42" H 4070 4696 50  0000 L CNN
 F 1 "178R" H 4070 4605 50  0000 L CNN
 F 2 "Resistor_SMD:R_0603_1608Metric" V 3930 4650 50  0001 C CNN
 F 3 "https://www.bourns.com/docs/product-datasheets/CRxxxxx.pdf" H 4000 4650 50  0001 C CNN
-F 4 "CR0603-FX-1780ELF" H 4000 4650 50  0001 C CNN "Part_number"
+F 4 "CR0603-FX-1780ELF" H 4000 4650 50  0001 C CNN "Part_number"
 	1    4000 4650
 	1    0    0    -1
@@
 AR Path="/603F1F4D/605BE11A/603E7162" Ref="D?"  Part="1"
 AR Path="/603F1F4D/605BE15A/603E7162" Ref="D?"  Part="1"
-F 0 "D9" H 5500 3697 50  0000 C CNN
+F 0 "D6" H 5500 3697 50  0000 C CNN
 F 1 "SMLVN6RGB1U" H 5500 3606 50  0000 C CNN
 F 2 "LitterRobot:ROHM_SMLVN6" H 5500 2850 50  0001 C CNN
@@
 AR Path="/603F1F4D/605BE11A/603FCE1E" Ref="R?"  Part="1"
 AR Path="/603F1F4D/605BE15A/603FCE1E" Ref="R?"  Part="1"
-F 0 "R52" H 5570 4696 50  0000 L CNN
+F 0 "R43" H 5570 4696 50  0000 L CNN
 F 1 "221R" H 5570 4605 50  0000 L CNN
 F 2 "Resistor_SMD:R_0603_1608Metric" V 5430 4650 50  0001 C CNN
@@
 AR Path="/603F1F4D/605BE11A/603FDBA6" Ref="R?"  Part="1"
 AR Path="/603F1F4D/605BE15A/603FDBA6" Ref="R?"  Part="1"
-F 0 "R53" H 7070 4696 50  0000 L CNN
+F 0 "R44" H 7070 4696 50  0000 L CNN
 F 1 "221R" H 7070 4605 50  0000 L CNN
 F 2 "Resistor_SMD:R_0603_1608Metric" V 6930 4650 50  0001 C CNN
@@
 AR Path="/603F1F4D/605BE11A/603FDE8C" Ref="#PWR?"  Part="1"
 AR Path="/603F1F4D/605BE15A/603FDE8C" Ref="#PWR?"  Part="1"
-F 0 "#PWR0120" H 4000 4750 50  0001 C CNN
+F 0 "#PWR0104" H 4000 4750 50  0001 C CNN
 F 1 "GND" H 4005 4827 50  0000 C CNN
 F 2 "" H 4000 5000 50  0001 C CNN
@@
 AR Path="/603F1F4D/605BE11A/603FF30B" Ref="#PWR?"  Part="1"
 AR Path="/603F1F4D/605BE15A/603FF30B" Ref="#PWR?"  Part="1"
-F 0 "#PWR0121" H 5500 4750 50  0001 C CNN
+F 0 "#PWR0105" H 5500 4750 50  0001 C CNN
 F 1 "GND" H 5505 4827 50  0000 C CNN
 F 2 "" H 5500 5000 50  0001 C CNN
@@
 AR Path="/603F1F4D/605BE11A/603FF5B6" Ref="#PWR?"  Part="1"
 AR Path="/603F1F4D/605BE15A/603FF5B6" Ref="#PWR?"  Part="1"
-F 0 "#PWR0122" H 7000 4750 50  0001 C CNN
+F 0 "#PWR0106" H 7000 4750 50  0001 C CNN
 F 1 "GND" H 7005 4827 50  0000 C CNN
 F 2 "" H 7000 5000 50  0001 C CNN
@@
 AR Path="/603F1F4D/605BE11A/60414150" Ref="#PWR?"  Part="1"
 AR Path="/603F1F4D/605BE15A/60414150" Ref="#PWR?"  Part="1"
-F 0 "#PWR0119" H 5500 1850 50  0001 C CNN
+F 0 "#PWR0103" H 5500 1850 50  0001 C CNN
 F 1 "+7V" H 5515 2173 50  0000 C CNN
 F 2 "" H 5500 2000 50  0001 C CNN
@@
 AR Path="/603F1F4D/605BE11A/6045060B" Ref="Q?"  Part="1"
 AR Path="/603F1F4D/605BE15A/6045060B" Ref="Q?"  Part="1"
-F 0 "Q20" H 5591 4246 50  0000 L CNN
+F 0 "Q11" H 5591 4246 50  0000 L CNN
 F 1 "BC817" H 5591 4155 50  0000 L CNN
 F 2 "Package_TO_SOT_SMD:SOT-23" H 5600 4125 50  0001 L CIN
@@
 AR Path="/603F1F4D/605BE11A/60450E24" Ref="Q?"  Part="1"
 AR Path="/603F1F4D/605BE15A/60450E24" Ref="Q?"  Part="1"
-F 0 "Q21" H 7091 4246 50  0000 L CNN
+F 0 "Q12" H 7091 4246 50  0000 L CNN
 F 1 "BC817" H 7091 4155 50  0000 L CNN
 F 2 "Package_TO_SOT_SMD:SOT-23" H 7100 4125 50  0001 L CIN

Commit message: Complete routing all signals
Changed lines of the file:
@@
 $Descr A4 11693 8268
 encoding utf-8
-Sheet 19 23
+Sheet 22 23
 Title "Litter Robot 3 - RGB LED"
 Date "2021-04-10"
@@
 AR Path="/603F1F4D/605BE11A/603E2469" Ref="Q?"  Part="1"
 AR Path="/603F1F4D/605BE15A/603E2469" Ref="Q?"  Part="1"
-F 0 "Q10" H 4091 4246 50  0000 L CNN
+F 0 "Q19" H 4091 4246 50  0000 L CNN
 F 1 "BC817" H 4091 4155 50  0000 L CNN
 F 2 "Package_TO_SOT_SMD:SOT-23" H 4100 4125 50  0001 L CIN
@@
 AR Path="/603F1F4D/605BE11A/603E246F" Ref="R?"  Part="1"
 AR Path="/603F1F4D/605BE15A/603E246F" Ref="R?"  Part="1"
-F 0 "R42" H 4070 4696 50  0000 L CNN
+F 0 "R51" H 4070 4696 50  0000 L CNN
 F 1 "178R" H 4070 4605 50  0000 L CNN
 F 2 "Resistor_SMD:R_0603_1608Metric" V 3930 4650 50  0001 C CNN
@@
 AR Path="/603F1F4D/605BE11A/603E7162" Ref="D?"  Part="1"
 AR Path="/603F1F4D/605BE15A/603E7162" Ref="D?"  Part="1"
-F 0 "D6" H 5500 3697 50  0000 C CNN
+F 0 "D9" H 5500 3697 50  0000 C CNN
 F 1 "SMLVN6RGB1U" H 5500 3606 50  0000 C CNN
 F 2 "LitterRobot:ROHM_SMLVN6" H 5500 2850 50  0001 C CNN
@@
 AR Path="/603F1F4D/605BE11A/603FCE1E" Ref="R?"  Part="1"
 AR Path="/603F1F4D/605BE15A/603FCE1E" Ref="R?"  Part="1"
-F 0 "R43" H 5570 4696 50  0000 L CNN
+F 0 "R52" H 5570 4696 50  0000 L CNN
 F 1 "221R" H 5570 4605 50  0000 L CNN
 F 2 "Resistor_SMD:R_0603_1608Metric" V 5430 4650 50  0001 C CNN
@@
 AR Path="/603F1F4D/605BE11A/603FDBA6" Ref="R?"  Part="1"
 AR Path="/603F1F4D/605BE15A/603FDBA6" Ref="R?"  Part="1"
-F 0 "R44" H 7070 4696 50  0000 L CNN
+F 0 "R53" H 7070 4696 50  0000 L CNN
 F 1 "221R" H 7070 4605 50  0000 L CNN
 F 2 "Resistor_SMD:R_0603_1608Metric" V 6930 4650 50  0001 C CNN
@@
 AR Path="/603F1F4D/605BE11A/603FDE8C" Ref="#PWR?"  Part="1"
 AR Path="/603F1F4D/605BE15A/603FDE8C" Ref="#PWR?"  Part="1"
-F 0 "#PWR0104" H 4000 4750 50  0001 C CNN
+F 0 "#PWR0120" H 4000 4750 50  0001 C CNN
 F 1 "GND" H 4005 4827 50  0000 C CNN
 F 2 "" H 4000 5000 50  0001 C CNN
@@
 AR Path="/603F1F4D/605BE11A/603FF30B" Ref="#PWR?"  Part="1"
 AR Path="/603F1F4D/605BE15A/603FF30B" Ref="#PWR?"  Part="1"
-F 0 "#PWR0105" H 5500 4750 50  0001 C CNN
+F 0 "#PWR0121" H 5500 4750 50  0001 C CNN
 F 1 "GND" H 5505 4827 50  0000 C CNN
 F 2 "" H 5500 5000 50  0001 C CNN
@@
 AR Path="/603F1F4D/605BE11A/603FF5B6" Ref="#PWR?"  Part="1"
 AR Path="/603F1F4D/605BE15A/603FF5B6" Ref="#PWR?"  Part="1"
-F 0 "#PWR0106" H 7000 4750 50  0001 C CNN
+F 0 "#PWR0122" H 7000 4750 50  0001 C CNN
 F 1 "GND" H 7005 4827 50  0000 C CNN
 F 2 "" H 7000 5000 50  0001 C CNN
@@
 AR Path="/603F1F4D/605BE11A/60414150" Ref="#PWR?"  Part="1"
 AR Path="/603F1F4D/605BE15A/60414150" Ref="#PWR?"  Part="1"
-F 0 "#PWR0103" H 5500 1850 50  0001 C CNN
+F 0 "#PWR0119" H 5500 1850 50  0001 C CNN
 F 1 "+7V" H 5515 2173 50  0000 C CNN
 F 2 "" H 5500 2000 50  0001 C CNN
@@
 AR Path="/603F1F4D/605BE11A/6045060B" Ref="Q?"  Part="1"
 AR Path="/603F1F4D/605BE15A/6045060B" Ref="Q?"  Part="1"
-F 0 "Q11" H 5591 4246 50  0000 L CNN
+F 0 "Q20" H 5591 4246 50  0000 L CNN
 F 1 "BC817" H 5591 4155 50  0000 L CNN
 F 2 "Package_TO_SOT_SMD:SOT-23" H 5600 4125 50  0001 L CIN
@@
 AR Path="/603F1F4D/605BE11A/60450E24" Ref="Q?"  Part="1"
 AR Path="/603F1F4D/605BE15A/60450E24" Ref="Q?"  Part="1"
-F 0 "Q12" H 7091 4246 50  0000 L CNN
+F 0 "Q21" H 7091 4246 50  0000 L CNN
 F 1 "BC817" H 7091 4155 50  0000 L CNN
 F 2 "Package_TO_SOT_SMD:SOT-23" H 7100 4125 50  0001 L CIN

Commit message: Export BOM
Changed lines of the file:
@@
 $Descr A4 11693 8268
 encoding utf-8
-Sheet 22 23
+Sheet 20 23
 Title "Litter Robot 3 - RGB LED"
 Date "2021-04-10"
@@
 AR Path="/603F1F4D/605BE11A/603E2469" Ref="Q?"  Part="1"
 AR Path="/603F1F4D/605BE15A/603E2469" Ref="Q?"  Part="1"
-F 0 "Q19" H 4091 4246 50  0000 L CNN
+F 0 "Q13" H 4091 4246 50  0000 L CNN
 F 1 "BC817" H 4091 4155 50  0000 L CNN
 F 2 "Package_TO_SOT_SMD:SOT-23" H 4100 4125 50  0001 L CIN
@@
 AR Path="/603F1F4D/605BE11A/603E246F" Ref="R?"  Part="1"
 AR Path="/603F1F4D/605BE15A/603E246F" Ref="R?"  Part="1"
-F 0 "R51" H 4070 4696 50  0000 L CNN
+F 0 "R45" H 4070 4696 50  0000 L CNN
 F 1 "178R" H 4070 4605 50  0000 L CNN
 F 2 "Resistor_SMD:R_0603_1608Metric" V 3930 4650 50  0001 C CNN
@@
 AR Path="/603F1F4D/605BE11A/603E7162" Ref="D?"  Part="1"
 AR Path="/603F1F4D/605BE15A/603E7162" Ref="D?"  Part="1"
-F 0 "D9" H 5500 3697 50  0000 C CNN
+F 0 "D7" H 5500 3697 50  0000 C CNN
 F 1 "SMLVN6RGB1U" H 5500 3606 50  0000 C CNN
 F 2 "LitterRobot:ROHM_SMLVN6" H 5500 2850 50  0001 C CNN
@@
 AR Path="/603F1F4D/605BE11A/603FCE1E" Ref="R?"  Part="1"
 AR Path="/603F1F4D/605BE15A/603FCE1E" Ref="R?"  Part="1"
-F 0 "R52" H 5570 4696 50  0000 L CNN
+F 0 "R46" H 5570 4696 50  0000 L CNN
 F 1 "221R" H 5570 4605 50  0000 L CNN
 F 2 "Resistor_SMD:R_0603_1608Metric" V 5430 4650 50  0001 C CNN
@@
 AR Path="/603F1F4D/605BE11A/603FDBA6" Ref="R?"  Part="1"
 AR Path="/603F1F4D/605BE15A/603FDBA6" Ref="R?"  Part="1"
-F 0 "R53" H 7070 4696 50  0000 L CNN
+F 0 "R47" H 7070 4696 50  0000 L CNN
 F 1 "221R" H 7070 4605 50  0000 L CNN
 F 2 "Resistor_SMD:R_0603_1608Metric" V 6930 4650 50  0001 C CNN
@@
 AR Path="/603F1F4D/605BE11A/603FDE8C" Ref="#PWR?"  Part="1"
 AR Path="/603F1F4D/605BE15A/603FDE8C" Ref="#PWR?"  Part="1"
-F 0 "#PWR0120" H 4000 4750 50  0001 C CNN
+F 0 "#PWR0108" H 4000 4750 50  0001 C CNN
 F 1 "GND" H 4005 4827 50  0000 C CNN
 F 2 "" H 4000 5000 50  0001 C CNN
@@
 AR Path="/603F1F4D/605BE11A/603FF30B" Ref="#PWR?"  Part="1"
 AR Path="/603F1F4D/605BE15A/603FF30B" Ref="#PWR?"  Part="1"
-F 0 "#PWR0121" H 5500 4750 50  0001 C CNN
+F 0 "#PWR0109" H 5500 4750 50  0001 C CNN
 F 1 "GND" H 5505 4827 50  0000 C CNN
 F 2 "" H 5500 5000 50  0001 C CNN
@@
 AR Path="/603F1F4D/605BE11A/603FF5B6" Ref="#PWR?"  Part="1"
 AR Path="/603F1F4D/605BE15A/603FF5B6" Ref="#PWR?"  Part="1"
-F 0 "#PWR0122" H 7000 4750 50  0001 C CNN
+F 0 "#PWR0110" H 7000 4750 50  0001 C CNN
 F 1 "GND" H 7005 4827 50  0000 C CNN
 F 2 "" H 7000 5000 50  0001 C CNN
@@
 AR Path="/603F1F4D/605BE11A/60414150" Ref="#PWR?"  Part="1"
 AR Path="/603F1F4D/605BE15A/60414150" Ref="#PWR?"  Part="1"
-F 0 "#PWR0119" H 5500 1850 50  0001 C CNN
+F 0 "#PWR0107" H 5500 1850 50  0001 C CNN
 F 1 "+7V" H 5515 2173 50  0000 C CNN
 F 2 "" H 5500 2000 50  0001 C CNN
@@
 AR Path="/603F1F4D/605BE11A/6045060B" Ref="Q?"  Part="1"
 AR Path="/603F1F4D/605BE15A/6045060B" Ref="Q?"  Part="1"
-F 0 "Q20" H 5591 4246 50  0000 L CNN
+F 0 "Q14" H 5591 4246 50  0000 L CNN
 F 1 "BC817" H 5591 4155 50  0000 L CNN
 F 2 "Package_TO_SOT_SMD:SOT-23" H 5600 4125 50  0001 L CIN
@@
 AR Path="/603F1F4D/605BE11A/60450E24" Ref="Q?"  Part="1"
 AR Path="/603F1F4D/605BE15A/60450E24" Ref="Q?"  Part="1"
-F 0 "Q21" H 7091 4246 50  0000 L CNN
+F 0 "Q15" H 7091 4246 50  0000 L CNN
 F 1 "BC817" H 7091 4155 50  0000 L CNN
 F 2 "Package_TO_SOT_SMD:SOT-23" H 7100 4125 50  0001 L CIN

Commit message: Add jumpers on the power supply outputs
Parts:
- renumbered R48 to R52, R49 to R53, R50 to R54
Changed lines of the file:
@@
 $Descr A4 11693 8268
 encoding utf-8
-Sheet 20 23
+Sheet 19 23
 Title "Litter Robot 3 - RGB LED"
-Date "2021-04-10"
+Date "2021-05-24"
 Rev "A1"
 Comp "L. Sartory"
@@
 AR Path="/603F1F4D/605BE11A/603E2469" Ref="Q?"  Part="1"
 AR Path="/603F1F4D/605BE15A/603E2469" Ref="Q?"  Part="1"
-F 0 "Q13" H 4091 4246 50  0000 L CNN
+F 0 "Q22" H 4091 4246 50  0000 L CNN
 F 1 "BC817" H 4091 4155 50  0000 L CNN
 F 2 "Package_TO_SOT_SMD:SOT-23" H 4100 4125 50  0001 L CIN
@@
 AR Path="/603E246F" Ref="R?"  Part="1"
 AR Path="/603E03AA/603E246F" Ref="R?"  Part="1"
-AR Path="/603E03AA/6040C394/603E246F" Ref="R48"  Part="1"
-AR Path="/603E03AA/6040F4A1/603E246F" Ref="R51"  Part="1"
-AR Path="/603E03AA/6040F5B7/603E246F" Ref="R54"  Part="1"
-AR Path="/603E03AA/603BF34F/603E246F" Ref="R39"  Part="1"
-AR Path="/603E03AA/603BF354/603E246F" Ref="R45"  Part="1"
-AR Path="/603E03AA/603BF359/603E246F" Ref="R42"  Part="1"
+AR Path="/603E03AA/6040C394/603E246F" Ref="R52"  Part="1"
+AR Path="/603E03AA/6040F4A1/603E246F" Ref="R55"  Part="1"
+AR Path="/603E03AA/6040F5B7/603E246F" Ref="R58"  Part="1"
+AR Path="/603E03AA/603BF34F/603E246F" Ref="R43"  Part="1"
+AR Path="/603E03AA/603BF354/603E246F" Ref="R49"  Part="1"
+AR Path="/603E03AA/603BF359/603E246F" Ref="R46"  Part="1"
 AR Path="/603E03AA/603BFBDC/603E246F" Ref="R?"  Part="1"
 AR Path="/603E03AA/603BFBE1/603E246F" Ref="R?"  Part="1"
 AR Path="/603E03AA/603BFBE6/603E246F" Ref="R?"  Part="1"
-AR Path="/603E03AA/603BFD93/603E246F" Ref="R36"  Part="1"
+AR Path="/603E03AA/603BFD93/603E246F" Ref="R40"  Part="1"
 AR Path="/603F1F4D/605BE101/603E246F" Ref="R?"  Part="1"
 AR Path="/603F1F4D/605BE106/603E246F" Ref="R?"  Part="1"
@@
 AR Path="/603F1F4D/605BE11A/603E246F" Ref="R?"  Part="1"
 AR Path="/603F1F4D/605BE15A/603E246F" Ref="R?"  Part="1"
-F 0 "R45" H 4070 4696 50  0000 L CNN
+F 0 "R58" H 4070 4696 50  0000 L CNN
 F 1 "178R" H 4070 4605 50  0000 L CNN
 F 2 "Resistor_SMD:R_0603_1608Metric" V 3930 4650 50  0001 C CNN
@@
 AR Path="/603F1F4D/605BE11A/603E7162" Ref="D?"  Part="1"
 AR Path="/603F1F4D/605BE15A/603E7162" Ref="D?"  Part="1"
-F 0 "D7" H 5500 3697 50  0000 C CNN
+F 0 "D10" H 5500 3697 50  0000 C CNN
 F 1 "SMLVN6RGB1U" H 5500 3606 50  0000 C CNN
 F 2 "LitterRobot:ROHM_SMLVN6" H 5500 2850 50  0001 C CNN
@@
 AR Path="/603FCE1E" Ref="R?"  Part="1"
 AR Path="/603E03AA/603FCE1E" Ref="R?"  Part="1"
-AR Path="/603E03AA/6040C394/603FCE1E" Ref="R49"  Part="1"
-AR Path="/603E03AA/6040F4A1/603FCE1E" Ref="R52"  Part="1"
-AR Path="/603E03AA/6040F5B7/603FCE1E" Ref="R55"  Part="1"
-AR Path="/603E03AA/603BF34F/603FCE1E" Ref="R40"  Part="1"
-AR Path="/603E03AA/603BF354/603FCE1E" Ref="R46"  Part="1"
-AR Path="/603E03AA/603BF359/603FCE1E" Ref="R43"  Part="1"
+AR Path="/603E03AA/6040C394/603FCE1E" Ref="R53"  Part="1"
+AR Path="/603E03AA/6040F4A1/603FCE1E" Ref="R56"  Part="1"
+AR Path="/603E03AA/6040F5B7/603FCE1E" Ref="R59"  Part="1"
+AR Path="/603E03AA/603BF34F/603FCE1E" Ref="R44"  Part="1"
+AR Path="/603E03AA/603BF354/603FCE1E" Ref="R50"  Part="1"
+AR Path="/603E03AA/603BF359/603FCE1E" Ref="R47"  Part="1"
 AR Path="/603E03AA/603BFBDC/603FCE1E" Ref="R?"  Part="1"
 AR Path="/603E03AA/603BFBE1/603FCE1E" Ref="R?"  Part="1"
 AR Path="/603E03AA/603BFBE6/603FCE1E" Ref="R?"  Part="1"
-AR Path="/603E03AA/603BFD93/603FCE1E" Ref="R37"  Part="1"
+AR Path="/603E03AA/603BFD93/603FCE1E" Ref="R41"  Part="1"
 AR Path="/603F1F4D/605BE101/603FCE1E" Ref="R?"  Part="1"
 AR Path="/603F1F4D/605BE106/603FCE1E" Ref="R?"  Part="1"
@@
 AR Path="/603F1F4D/605BE11A/603FCE1E" Ref="R?"  Part="1"
 AR Path="/603F1F4D/605BE15A/603FCE1E" Ref="R?"  Part="1"
-F 0 "R46" H 5570 4696 50  0000 L CNN
+F 0 "R59" H 5570 4696 50  0000 L CNN
 F 1 "221R" H 5570 4605 50  0000 L CNN
 F 2 "Resistor_SMD:R_0603_1608Metric" V 5430 4650 50  0001 C CNN
@@
 AR Path="/603FDBA6" Ref="R?"  Part="1"
 AR Path="/603E03AA/603FDBA6" Ref="R?"  Part="1"
-AR Path="/603E03AA/6040C394/603FDBA6" Ref="R50"  Part="1"
-AR Path="/603E03AA/6040F4A1/603FDBA6" Ref="R53"  Part="1"
-AR Path="/603E03AA/6040F5B7/603FDBA6" Ref="R56"  Part="1"
-AR Path="/603E03AA/603BF34F/603FDBA6" Ref="R41"  Part="1"
-AR Path="/603E03AA/603BF354/603FDBA6" Ref="R47"  Part="1"
-AR Path="/603E03AA/603BF359/603FDBA6" Ref="R44"  Part="1"
+AR Path="/603E03AA/6040C394/603FDBA6" Ref="R54"  Part="1"
+AR Path="/603E03AA/6040F4A1/603FDBA6" Ref="R57"  Part="1"
+AR Path="/603E03AA/6040F5B7/603FDBA6" Ref="R60"  Part="1"
+AR Path="/603E03AA/603BF34F/603FDBA6" Ref="R45"  Part="1"
+AR Path="/603E03AA/603BF354/603FDBA6" Ref="R51"  Part="1"
+AR Path="/603E03AA/603BF359/603FDBA6" Ref="R48"  Part="1"
 AR Path="/603E03AA/603BFBDC/603FDBA6" Ref="R?"  Part="1"
 AR Path="/603E03AA/603BFBE1/603FDBA6" Ref="R?"  Part="1"
 AR Path="/603E03AA/603BFBE6/603FDBA6" Ref="R?"  Part="1"
-AR Path="/603E03AA/603BFD93/603FDBA6" Ref="R38"  Part="1"
+AR Path="/603E03AA/603BFD93/603FDBA6" Ref="R42"  Part="1"
 AR Path="/603F1F4D/605BE101/603FDBA6" Ref="R?"  Part="1"
 AR Path="/603F1F4D/605BE106/603FDBA6" Ref="R?"  Part="1"
@@
 AR Path="/603F1F4D/605BE11A/603FDBA6" Ref="R?"  Part="1"
 AR Path="/603F1F4D/605BE15A/603FDBA6" Ref="R?"  Part="1"
-F 0 "R47" H 7070 4696 50  0000 L CNN
+F 0 "R60" H 7070 4696 50  0000 L CNN
 F 1 "221R" H 7070 4605 50  0000 L CNN
 F 2 "Resistor_SMD:R_0603_1608Metric" V 6930 4650 50  0001 C CNN
@@
 AR Path="/603F1F4D/605BE11A/603FDE8C" Ref="#PWR?"  Part="1"
 AR Path="/603F1F4D/605BE15A/603FDE8C" Ref="#PWR?"  Part="1"
-F 0 "#PWR0108" H 4000 4750 50  0001 C CNN
+F 0 "#PWR0120" H 4000 4750 50  0001 C CNN
 F 1 "GND" H 4005 4827 50  0000 C CNN
 F 2 "" H 4000 5000 50  0001 C CNN
@@
 AR Path="/603F1F4D/605BE11A/603FF30B" Ref="#PWR?"  Part="1"
 AR Path="/603F1F4D/605BE15A/603FF30B" Ref="#PWR?"  Part="1"
-F 0 "#PWR0109" H 5500 4750 50  0001 C CNN
+F 0 "#PWR0121" H 5500 4750 50  0001 C CNN
 F 1 "GND" H 5505 4827 50  0000 C CNN
 F 2 "" H 5500 5000 50  0001 C CNN
@@
 AR Path="/603F1F4D/605BE11A/603FF5B6" Ref="#PWR?"  Part="1"
 AR Path="/603F1F4D/605BE15A/603FF5B6" Ref="#PWR?"  Part="1"
-F 0 "#PWR0110" H 7000 4750 50  0001 C CNN
+F 0 "#PWR0122" H 7000 4750 50  0001 C CNN
 F 1 "GND" H 7005 4827 50  0000 C CNN
 F 2 "" H 7000 5000 50  0001 C CNN
@@
 AR Path="/603F1F4D/605BE11A/60414150" Ref="#PWR?"  Part="1"
 AR Path="/603F1F4D/605BE15A/60414150" Ref="#PWR?"  Part="1"
-F 0 "#PWR0107" H 5500 1850 50  0001 C CNN
+F 0 "#PWR0119" H 5500 1850 50  0001 C CNN
 F 1 "+7V" H 5515 2173 50  0000 C CNN
 F 2 "" H 5500 2000 50  0001 C CNN
@@
 AR Path="/603F1F4D/605BE11A/6045060B" Ref="Q?"  Part="1"
 AR Path="/603F1F4D/605BE15A/6045060B" Ref="Q?"  Part="1"
-F 0 "Q14" H 5591 4246 50  0000 L CNN
+F 0 "Q23" H 5591 4246 50  0000 L CNN
 F 1 "BC817" H 5591 4155 50  0000 L CNN
 F 2 "Package_TO_SOT_SMD:SOT-23" H 5600 4125 50  0001 L CIN
@@
 AR Path="/603F1F4D/605BE11A/60450E24" Ref="Q?"  Part="1"
 AR Path="/603F1F4D/605BE15A/60450E24" Ref="Q?"  Part="1"
-F 0 "Q15" H 7091 4246 50  0000 L CNN
+F 0 "Q24" H 7091 4246 50  0000 L CNN
 F 1 "BC817" H 7091 4155 50  0000 L CNN
 F 2 "Package_TO_SOT_SMD:SOT-23" H 7100 4125 50  0001 L CIN
