File: PCB/Bluetooth.sch (KiCad schematic (older format))
At the start: 1 part, among them U4 EMB1061

Commit message: Connect the Bluetooth module to the FPGA
Connections:
- net Bluetooth_CTS renamed Bluetooth_~CTS
- net Bluetooth_RTS renamed Bluetooth_~RTS
Changed lines of the file:
@@
 Bluetooth_RX
 Text HLabel 4000 3700 0    50   Output ~ 0
-Bluetooth_CTS
+Bluetooth_~CTS
 Text HLabel 4000 3600 0    50   Input ~ 0
-Bluetooth_RTS
+Bluetooth_~RTS
 Text HLabel 4000 3300 0    50   Input ~ 0
 Bluetooth_~RESET

Commit message: Fix invalid / missing part numbers
Parts:
- U4: Part_number (none) -> 113990637
Changed lines of the file:
@@
 F 2 "LitterRobot:MXCHIP_EMB1061" H 5500 3950 50  0001 C CNN
 F 3 "https://newwezhanhkoss.oss-cn-hongkong.aliyuncs.com/contents/sitefiles3603/18015345/files/22510..pdf?response-content-type=application%2Fpdf" H 5500 3950 50  0001 C CNN
+F 4 "113990637" H 5500 3400 50  0001 C CNN "Part_number"
 	1    5500 3400
 	1    0    0    -1
