File: PCB/FpgaPower.sch (KiCad schematic (older format))
At the start: 19 parts, among them U5 10CL016YE144C8G

Commit message: Cleaned up the schematics
Connections:
- net GND: now also U5.145 (EP)
Changed lines of the file:
@@
 encoding utf-8
 Sheet 19 19
-Title "FPGA power supply"
+Title "Litter Robot 3 - FPGA power supply"
 Date "2021-03-28"
 Rev "A1"
@@
 Text Notes 8500 3500 0    50   ~ 0
 +3V3 decoupling capacitors:\n1 per I/O bank
+$Comp
+L power:GND #PWR?
+U 1 1 607A4FF3
+P 5750 5750
+AR Path="/607A4FF3" Ref="#PWR?"  Part="1"
+AR Path="/60624089/607A4FF3" Ref="#PWR?"  Part="1"
+AR Path="/603F1F4D/607A4FF3" Ref="#PWR?"  Part="1"
+AR Path="/603F1F4D/60647CC2/607A4FF3" Ref="#PWR?"  Part="1"
+AR Path="/603F1F4D/60659E39/607A4FF3" Ref="#PWR0114"  Part="1"
+F 0 "#PWR0114" H 5750 5500 50  0001 C CNN
+F 1 "GND" H 5755 5577 50  0000 C CNN
+F 2 "" H 5750 5750 50  0001 C CNN
+F 3 "" H 5750 5750 50  0001 C CNN
+	1    5750 5750
+	1    0    0    -1
+$EndComp
+Wire Wire Line
+	5750 5750 5750 5650
 $EndSCHEMATC

Commit message: Plot the schematic as PDF
Parts:
- removed C24, C25, C26, C27, C28, C29, C30, C31: 100nF, Capacitor_SMD:C_0603_1608Metric, symbol Device:C
Other:
- note removed: "+3V3 decoupling capacitors:\n1 per I/O bank"

Commit message: Add support for the weight sensor
Parts:
- renumbered C14 to C20, C15 to C21, C16 to C22, C17 to C23, C18 to C24, C19 to C25, C20 to C26, C21 to C27, C22 to C28, C23 to C29, U5 to U4

Commit message: Add support for the hall sensors and dome LED
Parts:
- renumbered C20 to C23, C21 to C24, C22 to C25, C23 to C26, C24 to C27, C25 to C28, C26 to C29, C27 to C30, C28 to C31, C29 to C32, U4 to U5

Commit message: Re-annotate all components
Parts:
- renumbered C23 to C16, C25 to C17, C28 to C18, C31 to C19, C24 to C20, C26 to C21, C29 to C22, C32 to C23, C27 to C24, C30 to C25, U5 to U2
