File: PCB/HallSensors.sch (KiCad schematic (older format))
At the start: 9 parts, among them Q22 BSS138, Q23 BSS138, U4 MCP1700T-5002E/TT

Commit message: Re-annotate all components
Parts:
- renumbered C13 to C30, C14 to C31, Q22 to Q1, Q23 to Q2, R45 to R24, R47 to R25, R46 to R26, R48 to R27, U4 to U5
Changed lines of the file:
@@
 $Descr A4 11693 8268
 encoding utf-8
-Sheet 21 22
+Sheet 8 22
 Title "Litter Robot 3 - Hall sensors level shifters"
-Date "2021-04-03"
+Date "2021-04-05"
 Rev "A1"
 Comp "L. Sartory"
@@
 AR Path="/603F1DCE/606A6D92" Ref="#PWR?"  Part="1"
 AR Path="/60624089/606A6D92" Ref="#PWR?"  Part="1"
-AR Path="/60690B6B/606A6D92" Ref="#PWR074"  Part="1"
-F 0 "#PWR074" H 6250 3250 50  0001 C CNN
+AR Path="/60690B6B/606A6D92" Ref="#PWR077"  Part="1"
+F 0 "#PWR077" H 6250 3250 50  0001 C CNN
 F 1 "+3V3" H 6265 3573 50  0000 C CNN
 F 2 "" H 6250 3400 50  0001 C CNN
@@
 AR Path="/603F1DCE/606AB6F0" Ref="#PWR?"  Part="1"
 AR Path="/60624089/606AB6F0" Ref="#PWR?"  Part="1"
-AR Path="/60690B6B/606AB6F0" Ref="#PWR075"  Part="1"
-F 0 "#PWR075" H 6250 4750 50  0001 C CNN
+AR Path="/60690B6B/606AB6F0" Ref="#PWR078"  Part="1"
+F 0 "#PWR078" H 6250 4750 50  0001 C CNN
 F 1 "+3V3" H 6265 5073 50  0000 C CNN
 F 2 "" H 6250 4900 50  0001 C CNN
@@
 AR Path="/603F1DCE/606C5787" Ref="#PWR?"  Part="1"
 AR Path="/60624089/606C5787" Ref="#PWR?"  Part="1"
-AR Path="/60690B6B/606C5787" Ref="#PWR072"  Part="1"
-F 0 "#PWR072" H 4500 1750 50  0001 C CNN
+AR Path="/60690B6B/606C5787" Ref="#PWR075"  Part="1"
+F 0 "#PWR075" H 4500 1750 50  0001 C CNN
 F 1 "+7V" H 4515 2073 50  0000 C CNN
 F 2 "" H 4500 1900 50  0001 C CNN
@@
 AR Path="/603F1DCE/606A5BB1" Ref="R?"  Part="1"
 AR Path="/60624089/606A5BB1" Ref="R?"  Part="1"
-AR Path="/60690B6B/606A5BB1" Ref="R47"  Part="1"
-F 0 "R47" H 6320 3796 50  0000 L CNN
+AR Path="/60690B6B/606A5BB1" Ref="R25"  Part="1"
+F 0 "R25" H 6320 3796 50  0000 L CNN
 F 1 "10k" H 6320 3705 50  0000 L CNN
 F 2 "Resistor_SMD:R_0603_1608Metric" V 6180 3750 50  0001 C CNN
@@
 AR Path="/603F1DCE/606A5B75" Ref="R?"  Part="1"
 AR Path="/60624089/606A5B75" Ref="R?"  Part="1"
-AR Path="/60690B6B/606A5B75" Ref="R45"  Part="1"
-F 0 "R45" H 5320 3796 50  0000 L CNN
+AR Path="/60690B6B/606A5B75" Ref="R24"  Part="1"
+F 0 "R24" H 5320 3796 50  0000 L CNN
 F 1 "10k" H 5320 3705 50  0000 L CNN
 F 2 "Resistor_SMD:R_0603_1608Metric" V 5180 3750 50  0001 C CNN
@@
 AR Path="/603F1DCE/606AB6EA" Ref="R?"  Part="1"
 AR Path="/60624089/606AB6EA" Ref="R?"  Part="1"
-AR Path="/60690B6B/606AB6EA" Ref="R48"  Part="1"
-F 0 "R48" H 6320 5296 50  0000 L CNN
+AR Path="/60690B6B/606AB6EA" Ref="R27"  Part="1"
+F 0 "R27" H 6320 5296 50  0000 L CNN
 F 1 "10k" H 6320 5205 50  0000 L CNN
 F 2 "Resistor_SMD:R_0603_1608Metric" V 6180 5250 50  0001 C CNN
@@
 AR Path="/603F1DCE/606AB6E3" Ref="R?"  Part="1"
 AR Path="/60624089/606AB6E3" Ref="R?"  Part="1"
-AR Path="/60690B6B/606AB6E3" Ref="R46"  Part="1"
-F 0 "R46" H 5320 5296 50  0000 L CNN
+AR Path="/60690B6B/606AB6E3" Ref="R26"  Part="1"
+F 0 "R26" H 5320 5296 50  0000 L CNN
 F 1 "10k" H 5320 5205 50  0000 L CNN
 F 2 "Resistor_SMD:R_0603_1608Metric" V 5180 5250 50  0001 C CNN
@@
 $EndComp
 $Comp
-L Transistor_FET:BSS138 Q22
+L Transistor_FET:BSS138 Q1
 U 1 1 606D0473
 P 5750 3900
-F 0 "Q22" V 5999 3900 50  0000 C CNN
+F 0 "Q1" V 5999 3900 50  0000 C CNN
 F 1 "BSS138" V 6090 3900 50  0000 C CNN
 F 2 "Package_TO_SOT_SMD:SOT-23" H 5950 3825 50  0001 L CIN
@@
 $EndComp
 $Comp
-L Transistor_FET:BSS138 Q23
+L Transistor_FET:BSS138 Q2
 U 1 1 606D7597
 P 5750 5400
-F 0 "Q23" V 5999 5400 50  0000 C CNN
+F 0 "Q2" V 5999 5400 50  0000 C CNN
 F 1 "BSS138" V 6090 5400 50  0000 C CNN
 F 2 "Package_TO_SOT_SMD:SOT-23" H 5950 5325 50  0001 L CIN
@@
 $EndComp
 $Comp
-L Regulator_Linear:MCP1700-5002E_SOT23 U4
+L Regulator_Linear:MCP1700-5002E_SOT23 U5
 U 1 1 606E41AA
 P 5250 2000
-F 0 "U4" H 5250 2242 50  0000 C CNN
+F 0 "U5" H 5250 2242 50  0000 C CNN
 F 1 "MCP1700T-5002E/TT" H 5250 2151 50  0000 C CNN
 F 2 "Package_TO_SOT_SMD:SOT-23" H 5250 2225 50  0001 C CNN
@@
 P 5250 2600
 AR Path="/606E736A" Ref="#PWR?"  Part="1"
-AR Path="/60690B6B/606E736A" Ref="#PWR073"  Part="1"
-F 0 "#PWR073" H 5250 2350 50  0001 C CNN
+AR Path="/60690B6B/606E736A" Ref="#PWR076"  Part="1"
+F 0 "#PWR076" H 5250 2350 50  0001 C CNN
 F 1 "GND" H 5255 2427 50  0000 C CNN
 F 2 "" H 5250 2600 50  0001 C CNN
@@
 AR Path="/603F1DCE/606F23E8" Ref="C?"  Part="1"
 AR Path="/60624089/606F23E8" Ref="C?"  Part="1"
-AR Path="/60690B6B/606F23E8" Ref="C14"  Part="1"
-F 0 "C14" H 6115 2341 50  0000 L CNN
+AR Path="/60690B6B/606F23E8" Ref="C31"  Part="1"
+F 0 "C31" H 6115 2341 50  0000 L CNN
 F 1 "1µF" H 6115 2250 50  0000 L CNN
 F 2 "Capacitor_SMD:C_0603_1608Metric" H 6038 2100 50  0001 C CNN
@@
 AR Path="/603F1DCE/606F762A" Ref="C?"  Part="1"
 AR Path="/60624089/606F762A" Ref="C?"  Part="1"
-AR Path="/60690B6B/606F762A" Ref="C13"  Part="1"
-F 0 "C13" H 4615 2341 50  0000 L CNN
+AR Path="/60690B6B/606F762A" Ref="C30"  Part="1"
+F 0 "C30" H 4615 2341 50  0000 L CNN
 F 1 "1µF" H 4615 2250 50  0000 L CNN
 F 2 "Capacitor_SMD:C_0603_1608Metric" H 4538 2100 50  0001 C CNN

Commit message: Add the EMB1061 Bluetooth module
Parts:
- renumbered U5 to U6
Changed lines of the file:
@@
 $Descr A4 11693 8268
 encoding utf-8
-Sheet 8 22
+Sheet 8 23
 Title "Litter Robot 3 - Hall sensors level shifters"
-Date "2021-04-05"
+Date "2021-04-10"
 Rev "A1"
 Comp "L. Sartory"
@@
 AR Path="/603F1DCE/606A6D92" Ref="#PWR?"  Part="1"
 AR Path="/60624089/606A6D92" Ref="#PWR?"  Part="1"
-AR Path="/60690B6B/606A6D92" Ref="#PWR077"  Part="1"
-F 0 "#PWR077" H 6250 3250 50  0001 C CNN
+AR Path="/60690B6B/606A6D92" Ref="#PWR080"  Part="1"
+F 0 "#PWR080" H 6250 3250 50  0001 C CNN
 F 1 "+3V3" H 6265 3573 50  0000 C CNN
 F 2 "" H 6250 3400 50  0001 C CNN
@@
 AR Path="/603F1DCE/606AB6F0" Ref="#PWR?"  Part="1"
 AR Path="/60624089/606AB6F0" Ref="#PWR?"  Part="1"
-AR Path="/60690B6B/606AB6F0" Ref="#PWR078"  Part="1"
-F 0 "#PWR078" H 6250 4750 50  0001 C CNN
+AR Path="/60690B6B/606AB6F0" Ref="#PWR081"  Part="1"
+F 0 "#PWR081" H 6250 4750 50  0001 C CNN
 F 1 "+3V3" H 6265 5073 50  0000 C CNN
 F 2 "" H 6250 4900 50  0001 C CNN
@@
 AR Path="/603F1DCE/606C5787" Ref="#PWR?"  Part="1"
 AR Path="/60624089/606C5787" Ref="#PWR?"  Part="1"
-AR Path="/60690B6B/606C5787" Ref="#PWR075"  Part="1"
-F 0 "#PWR075" H 4500 1750 50  0001 C CNN
+AR Path="/60690B6B/606C5787" Ref="#PWR078"  Part="1"
+F 0 "#PWR078" H 4500 1750 50  0001 C CNN
 F 1 "+7V" H 4515 2073 50  0000 C CNN
 F 2 "" H 4500 1900 50  0001 C CNN
@@
 $EndComp
 $Comp
-L Regulator_Linear:MCP1700-5002E_SOT23 U5
+L Regulator_Linear:MCP1700-5002E_SOT23 U6
 U 1 1 606E41AA
 P 5250 2000
-F 0 "U5" H 5250 2242 50  0000 C CNN
+F 0 "U6" H 5250 2242 50  0000 C CNN
 F 1 "MCP1700T-5002E/TT" H 5250 2151 50  0000 C CNN
 F 2 "Package_TO_SOT_SMD:SOT-23" H 5250 2225 50  0001 C CNN
@@
 P 5250 2600
 AR Path="/606E736A" Ref="#PWR?"  Part="1"
-AR Path="/60690B6B/606E736A" Ref="#PWR076"  Part="1"
-F 0 "#PWR076" H 5250 2350 50  0001 C CNN
+AR Path="/60690B6B/606E736A" Ref="#PWR079"  Part="1"
+F 0 "#PWR079" H 5250 2350 50  0001 C CNN
 F 1 "GND" H 5255 2427 50  0000 C CNN
 F 2 "" H 5250 2600 50  0001 C CNN

Commit message: Add jumpers on the power supply outputs
Parts:
- renumbered R24 to R28, R25 to R29, R26 to R30, R27 to R31
Changed lines of the file:
@@
 Sheet 9 23
 Title "Litter Robot 3 - Hall sensors level shifters"
-Date "2021-04-10"
+Date "2021-05-24"
 Rev "A1"
 Comp "L. Sartory"
@@
 AR Path="/603F1DCE/606A5BB1" Ref="R?"  Part="1"
 AR Path="/60624089/606A5BB1" Ref="R?"  Part="1"
-AR Path="/60690B6B/606A5BB1" Ref="R25"  Part="1"
-F 0 "R25" H 6320 3796 50  0000 L CNN
+AR Path="/60690B6B/606A5BB1" Ref="R29"  Part="1"
+F 0 "R29" H 6320 3796 50  0000 L CNN
 F 1 "10k" H 6320 3705 50  0000 L CNN
 F 2 "Resistor_SMD:R_0603_1608Metric" V 6180 3750 50  0001 C CNN
@@
 AR Path="/603F1DCE/606A5B75" Ref="R?"  Part="1"
 AR Path="/60624089/606A5B75" Ref="R?"  Part="1"
-AR Path="/60690B6B/606A5B75" Ref="R24"  Part="1"
-F 0 "R24" H 5320 3796 50  0000 L CNN
+AR Path="/60690B6B/606A5B75" Ref="R28"  Part="1"
+F 0 "R28" H 5320 3796 50  0000 L CNN
 F 1 "10k" H 5320 3705 50  0000 L CNN
 F 2 "Resistor_SMD:R_0603_1608Metric" V 5180 3750 50  0001 C CNN
@@
 AR Path="/603F1DCE/606AB6EA" Ref="R?"  Part="1"
 AR Path="/60624089/606AB6EA" Ref="R?"  Part="1"
-AR Path="/60690B6B/606AB6EA" Ref="R27"  Part="1"
-F 0 "R27" H 6320 5296 50  0000 L CNN
+AR Path="/60690B6B/606AB6EA" Ref="R31"  Part="1"
+F 0 "R31" H 6320 5296 50  0000 L CNN
 F 1 "10k" H 6320 5205 50  0000 L CNN
 F 2 "Resistor_SMD:R_0603_1608Metric" V 6180 5250 50  0001 C CNN
@@
 AR Path="/603F1DCE/606AB6E3" Ref="R?"  Part="1"
 AR Path="/60624089/606AB6E3" Ref="R?"  Part="1"
-AR Path="/60690B6B/606AB6E3" Ref="R26"  Part="1"
-F 0 "R26" H 5320 5296 50  0000 L CNN
+AR Path="/60690B6B/606AB6E3" Ref="R30"  Part="1"
+F 0 "R30" H 5320 5296 50  0000 L CNN
 F 1 "10k" H 5320 5205 50  0000 L CNN
 F 2 "Resistor_SMD:R_0603_1608Metric" V 5180 5250 50  0001 C CNN
